Commit message: update for use with reach

File: jackal_launch/urdf/jackal_mods.urdf.xacro (robot description, xacro)
@@ -1,6 +1,6 @@
 <?xml version="1.0"?>
 <robot xmlns:xacro="http://www.ros.org/wiki/xacro">
-  <link name="piksi_link">
-    <!--Piksi antena-->
+  <link name="read_link">
+    <!--reach antena-->
     <visual>
       <geometry>
@@ -27,7 +27,7 @@
     </visual>
   </link>
-  <joint name="piksi_joint" type="fixed">
+  <joint name="reach_joint" type="fixed">
     <parent link="chassis_link" />
-    <child link="piksi_link" />
+    <child link="reach_link" />
     <origin xyz="-0.190 -0.12 0.60" />
   </joint>

Commit message: fix stuff

File: jackal_launch/urdf/jackal_mods.urdf.xacro (robot description, xacro)
@@ -1,5 +1,5 @@
 <?xml version="1.0"?>
 <robot xmlns:xacro="http://www.ros.org/wiki/xacro">
-  <link name="read_link">
+  <link name="reach_link">
     <!--reach antena-->
     <visual>
